File: project/intelliputer_connector.kicad_pcb (KiCad board)
At the start: 2 copper layers, 68.1 x 83.9 mm, 2 parts, among them J1 44-contact card edge, J2 Ribbon header, 2x22, 2.54 mm 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

Commit message: Finalize precision edge connector production package
Other:
- board text added: "01 GND"
- board text added: "02 GND/VID"
- board text added: "03 ~MSYNC"
- board text added: "04 CBLNK"
- board text added: "05 DB7"
- board text added: "06 EXT AUD"
- board text added: "07 DB8"
- board text added: "08 EXT VID"
- board text added: "09 DB6"
- board text added: "10 MCLK"
- board text added: "11 DB9"
- board text added: "12 RESET"
- board text added: "13 DB5"
- board text added: "14 SR1"
- board text added: "15 DB10"
- board text added: "16 SER OUT"
- board text added: "17 DB4"
- board text added: "18 SER IN"
- board text added: "19 DB11"
- board text added: "20 ROM DIS"
- board text added: "21 DB3"
- board text added: "22 GND"
- board text added: "23 DB12"
- board text added: "24 GND"
- board text added: "25 DB13"
- board text added: "26 GND"
- board text added: "27 DB2"
- board text added: "28 GND"
- board text added: "29 DB14"
- board text added: "30 ~BUSAK"
- board text added: "31 DB1"
- board text added: "32 BC1 IN"
- board text added: "33 DB0"
- board text added: "34 BC2 IN"
- board text added: "35 DB15"
- board text added: "36 BDIR IN"
- board text added: "37 BDIR OUT"
- board text added: "38 BDIR OUT"
- board text added: "39 BC2 OUT"
- board text added: "40 BC2 OUT"
- board text added: "41 BC1 OUT"
- board text added: "42 BC1 OUT"
- board text added: "43 +5V"
- board text added: "44 GND"
- board text added: "CARTRIDGE PORT PIN ASSIGNMENTS"
- board text removed: "01 GND / 02 GND/VID"
- board text removed: "03 ~MSYNC / 04 CBLNK"
- board text removed: "05 DB7 / 06 EXT AUD"
- board text removed: "07 DB8 / 08 EXT VID"
- board text removed: "09 DB6 / 10 MCLK"
- board text removed: "11 DB9 / 12 RESET"
- board text removed: "13 DB5 / 14 SR1"
- board text removed: "15 DB10 / 16 SER OUT"
- board text removed: "17 DB4 / 18 SER IN"
- board text removed: "19 DB11 / 20 ROM DIS"
- board text removed: "21 DB3 / 22 GND"
- board text removed: "23 DB12 / 24 GND"
- board text removed: "25 DB13 / 26 GND"
- board text removed: "27 DB2 / 28 GND"
- board text removed: "29 DB14 / 30 ~BUSAK"
- board text removed: "31 DB1 / 32 BC1 IN"
- board text removed: "33 DB0 / 34 BC2 IN"
- board text removed: "35 DB15 / 36 BDIR IN"
- board text removed: "37 BDIR OUT / 38 BDIR OUT"
- board text removed: "39 BC2 OUT / 40 BC2 OUT"
- board text removed: "41 BC1 OUT / 42 BC1 OUT"
- board text removed: "43 +5V / 44 GND"
Changed lines of the file:
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@@
 	(generator_version "10.0")
 	(general
-		(thickness 1.6)
+		(thickness 1.55)
 		(legacy_teardrops no)
 	)
@@
 		)
 	)
-	(gr_text "01 GND / 02 GND/VID" (at 133 132 0) (layer "B.SilkS") (effects (font (size 0.8 0.8) (thickness 0.12)) (justify mirror)))
-	(gr_text "03 ~MSYNC / 04 CBLNK" (at 133 133.6 0) (layer "B.SilkS") (effects (font (size 0.8 0.8) (thickness 0.12)) (justify mirror)))
-	(gr_text "05 DB7 / 06 EXT AUD" (at 133 135.2 0) (layer "B.SilkS") (effects (font (size 0.8 0.8) (thickness 0.12)) (justify mirror)))
-	(gr_text "07 DB8 / 08 EXT VID" (at 133 136.8 0) (layer "B.SilkS") (effects (font (size 0.8 0.8) (thickness 0.12)) (justify mirror)))
-	(gr_text "09 DB6 / 10 MCLK" (at 133 138.4 0) (layer "B.SilkS") (effects (font (size 0.8 0.8) (thickness 0.12)) (justify mirror)))
-	(gr_text "11 DB9 / 12 RESET" (at 133 140 0) (layer "B.SilkS") (effects (font (size 0.8 0.8) (thickness 0.12)) (justify mirror)))
-	(gr_text "13 DB5 / 14 SR1" (at 133 141.6 0) (layer "B.SilkS") (effects (font (size 0.8 0.8) (thickness 0.12)) (justify mirror)))
-	(gr_text "15 DB10 / 16 SER OUT" (at 133 143.2 0) (layer "B.SilkS") (effects (font (size 0.8 0.8) (thickness 0.12)) (justify mirror)))
-	(gr_text "17 DB4 / 18 SER IN" (at 133 144.8 0) (layer "B.SilkS") (effects (font (size 0.8 0.8) (thickness 0.12)) (justify mirror)))
-	(gr_text "19 DB11 / 20 ROM DIS" (at 133 146.4 0) (layer "B.SilkS") (effects (font (size 0.8 0.8) (thickness 0.12)) (justify mirror)))
-	(gr_text "21 DB3 / 22 GND" (at 133 148 0) (layer "B.SilkS") (effects (font (size 0.8 0.8) (thickness 0.12)) (justify mirror)))
-	(gr_text "23 DB12 / 24 GND" (at 103 132 0) (layer "B.SilkS") (effects (font (size 0.8 0.8) (thickness 0.12)) (justify mirror)))
-	(gr_text "25 DB13 / 26 GND" (at 103 133.6 0) (layer "B.SilkS") (effects (font (size 0.8 0.8) (thickness 0.12)) (justify mirror)))
-	(gr_text "27 DB2 / 28 GND" (at 103 135.2 0) (layer "B.SilkS") (effects (font (size 0.8 0.8) (thickness 0.12)) (justify mirror)))
-	(gr_text "29 DB14 / 30 ~BUSAK" (at 103 136.8 0) (layer "B.SilkS") (effects (font (size 0.8 0.8) (thickness 0.12)) (justify mirror)))
-	(gr_text "31 DB1 / 32 BC1 IN" (at 103 138.4 0) (layer "B.SilkS") (effects (font (size 0.8 0.8) (thickness 0.12)) (justify mirror)))
-	(gr_text "33 DB0 / 34 BC2 IN" (at 103 140 0) (layer "B.SilkS") (effects (font (size 0.8 0.8) (thickness 0.12)) (justify mirror)))
-	(gr_text "35 DB15 / 36 BDIR IN" (at 103 141.6 0) (layer "B.SilkS") (effects (font (size 0.8 0.8) (thickness 0.12)) (justify mirror)))
-	(gr_text "37 BDIR OUT / 38 BDIR OUT" (at 103 143.2 0) (layer "B.SilkS") (effects (font (size 0.8 0.8) (thickness 0.12)) (justify mirror)))
-	(gr_text "39 BC2 OUT / 40 BC2 OUT" (at 103 144.8 0) (layer "B.SilkS") (effects (font (size 0.8 0.8) (thickness 0.12)) (justify mirror)))
-	(gr_text "41 BC1 OUT / 42 BC1 OUT" (at 103 146.4 0) (layer "B.SilkS") (effects (font (size 0.8 0.8) (thickness 0.12)) (justify mirror)))
-	(gr_text "43 +5V / 44 GND" (at 103 148 0) (layer "B.SilkS") (effects (font (size 0.8 0.8) (thickness 0.12)) (justify mirror)))
+	(gr_text "01 GND" (at 135.5 132 0) (layer "B.SilkS") (effects (font (size 0.8 0.8) (thickness 0.12)) (justify mirror right)))
+	(gr_text "03 ~MSYNC" (at 135.5 133.6 0) (layer "B.SilkS") (effects (font (size 0.8 0.8) (thickness 0.12)) (justify mirror right)))
+	(gr_text "05 DB7" (at 135.5 135.2 0) (layer "B.SilkS") (effects (font (size 0.8 0.8) (thickness 0.12)) (justify mirror right)))
+	(gr_text "07 DB8" (at 135.5 136.8 0) (layer "B.SilkS") (effects (font (size 0.8 0.8) (thickness 0.12)) (justify mirror right)))
+	(gr_text "09 DB6" (at 135.5 138.4 0) (layer "B.SilkS") (effects (font (size 0.8 0.8) (thickness 0.12)) (justify mirror right)))
+	(gr_text "11 DB9" (at 135.5 140 0) (layer "B.SilkS") (effects (font (size 0.8 0.8) (thickness 0.12)) (justify mirror right)))
+	(gr_text "13 DB5" (at 135.5 141.6 0) (layer "B.SilkS") (effects (font (size 0.8 0.8) (thickness 0.12)) (justify mirror right)))
+	(gr_text "15 DB10" (at 135.5 143.2 0) (layer "B.SilkS") (effects (font (size 0.8 0.8) (thickness 0.12)) (justify mirror right)))
+	(gr_text "17 DB4" (at 135.5 144.8 0) (layer "B.SilkS") (effects (font (size 0.8 0.8) (thickness 0.12)) (justify mirror right)))
+	(gr_text "19 DB11" (at 135.5 146.4 0) (layer "B.SilkS") (effects (font (size 0.8 0.8) (thickness 0.12)) (justify mirror right)))
+	(gr_text "21 DB3" (at 135.5 148 0) (layer "B.SilkS") (effects (font (size 0.8 0.8) (thickness 0.12)) (justify mirror right)))
+	(gr_text "23 DB12" (at 104.9 132 0) (layer "B.SilkS") (effects (font (size 0.8 0.8) (thickness 0.12)) (justify mirror right)))
+	(gr_text "25 DB13" (at 104.9 133.6 0) (layer "B.SilkS") (effects (font (size 0.8 0.8) (thickness 0.12)) (justify mirror right)))
+	(gr_text "27 DB2" (at 104.9 135.2 0) (layer "B.SilkS") (effects (font (size 0.8 0.8) (thickness 0.12)) (justify mirror right)))
+	(gr_text "29 DB14" (at 104.9 136.8 0) (layer "B.SilkS") (effects (font (size 0.8 0.8) (thickness 0.12)) (justify mirror right)))
+	(gr_text "31 DB1" (at 104.9 138.4 0) (layer "B.SilkS") (effects (font (size 0.8 0.8) (thickness 0.12)) (justify mirror right)))
+	(gr_text "33 DB0" (at 104.9 140 0) (layer "B.SilkS") (effects (font (size 0.8 0.8) (thickness 0.12)) (justify mirror right)))
+	(gr_text "35 DB15" (at 104.9 141.6 0) (layer "B.SilkS") (effects (font (size 0.8 0.8) (thickness 0.12)) (justify mirror right)))
+	(gr_text "37 BDIR OUT" (at 104.9 143.2 0) (layer "B.SilkS") (effects (font (size 0.8 0.8) (thickness 0.12)) (justify mirror right)))
+	(gr_text "39 BC2 OUT" (at 104.9 144.8 0) (layer "B.SilkS") (effects (font (size 0.8 0.8) (thickness 0.12)) (justify mirror right)))
+	(gr_text "41 BC1 OUT" (at 104.9 146.4 0) (layer "B.SilkS") (effects (font (size 0.8 0.8) (thickness 0.12)) (justify mirror right)))
+	(gr_text "43 +5V" (at 104.9 148 0) (layer "B.SilkS") (effects (font (size 0.8 0.8) (thickness 0.12)) (justify mirror right)))
+	(gr_text "02 GND/VID" (at 134.7 132 0) (layer "B.SilkS") (effects (font (size 0.8 0.8) (thickness 0.12)) (justify mirror left)))
+	(gr_text "04 CBLNK" (at 134.7 133.6 0) (layer "B.SilkS") (effects (font (size 0.8 0.8) (thickness 0.12)) (justify mirror left)))
+	(gr_text "06 EXT AUD" (at 134.7 135.2 0) (layer "B.SilkS") (effects (font (size 0.8 0.8) (thickness 0.12)) (justify mirror left)))
+	(gr_text "08 EXT VID" (at 134.7 136.8 0) (layer "B.SilkS") (effects (font (size 0.8 0.8) (thickness 0.12)) (justify mirror left)))
+	(gr_text "10 MCLK" (at 134.7 138.4 0) (layer "B.SilkS") (effects (font (size 0.8 0.8) (thickness 0.12)) (justify mirror left)))
+	(gr_text "12 RESET" (at 134.7 140 0) (layer "B.SilkS") (effects (font (size 0.8 0.8) (thickness 0.12)) (justify mirror left)))
+	(gr_text "14 SR1" (at 134.7 141.6 0) (layer "B.SilkS") (effects (font (size 0.8 0.8) (thickness 0.12)) (justify mirror left)))
+	(gr_text "16 SER OUT" (at 134.7 143.2 0) (layer "B.SilkS") (effects (font (size 0.8 0.8) (thickness 0.12)) (justify mirror left)))
+	(gr_text "18 SER IN" (at 134.7 144.8 0) (layer "B.SilkS") (effects (font (size 0.8 0.8) (thickness 0.12)) (justify mirror left)))
+	(gr_text "20 ROM DIS" (at 134.7 146.4 0) (layer "B.SilkS") (effects (font (size 0.8 0.8) (thickness 0.12)) (justify mirror left)))
+	(gr_text "22 GND" (at 134.7 148 0) (layer "B.SilkS") (effects (font (size 0.8 0.8) (thickness 0.12)) (justify mirror left)))
+	(gr_text "24 GND" (at 104.3 132 0) (layer "B.SilkS") (effects (font (size 0.8 0.8) (thickness 0.12)) (justify mirror left)))
+	(gr_text "26 GND" (at 104.3 133.6 0) (layer "B.SilkS") (effects (font (size 0.8 0.8) (thickness 0.12)) (justify mirror left)))
+	(gr_text "28 GND" (at 104.3 135.2 0) (layer "B.SilkS") (effects (font (size 0.8 0.8) (thickness 0.12)) (justify mirror left)))
+	(gr_text "30 ~BUSAK" (at 104.3 136.8 0) (layer "B.SilkS") (effects (font (size 0.8 0.8) (thickness 0.12)) (justify mirror left)))
+	(gr_text "32 BC1 IN" (at 104.3 138.4 0) (layer "B.SilkS") (effects (font (size 0.8 0.8) (thickness 0.12)) (justify mirror left)))
+	(gr_text "34 BC2 IN" (at 104.3 140 0) (layer "B.SilkS") (effects (font (size 0.8 0.8) (thickness 0.12)) (justify mirror left)))
+	(gr_text "36 BDIR IN" (at 104.3 141.6 0) (layer "B.SilkS") (effects (font (size 0.8 0.8) (thickness 0.12)) (justify mirror left)))
+	(gr_text "38 BDIR OUT" (at 104.3 143.2 0) (layer "B.SilkS") (effects (font (size 0.8 0.8) (thickness 0.12)) (justify mirror left)))
+	(gr_text "40 BC2 OUT" (at 104.3 144.8 0) (layer "B.SilkS") (effects (font (size 0.8 0.8) (thickness 0.12)) (justify mirror left)))
+	(gr_text "42 BC1 OUT" (at 104.3 146.4 0) (layer "B.SilkS") (effects (font (size 0.8 0.8) (thickness 0.12)) (justify mirror left)))
+	(gr_text "44 GND" (at 104.3 148 0) (layer "B.SilkS") (effects (font (size 0.8 0.8) (thickness 0.12)) (justify mirror left)))
+	(gr_line (start 135.1 131.2) (end 135.1 148.8) (stroke (width 0.12) (type solid)) (layer "B.SilkS"))
+	(gr_line (start 104.5 131.2) (end 104.5 148.8) (stroke (width 0.12) (type solid)) (layer "B.SilkS"))
+	(gr_text "CARTRIDGE PORT PIN ASSIGNMENTS" (at 118 126 0) (layer "B.SilkS") (effects (font (size 1.0 1.0) (thickness 0.15)) (justify mirror)))
 	(gr_text "INTELLIPUTER CONNECTOR"
 		(at 118 117.5 0)
